File: pmod_sram/pmod_sram.kicad_sch (KiCad schematic)
At the start: 4 parts, among them J1 PMOD connector, U1 23LC1024 (SOIC8)

Commit message: New versions of PCB
Parts:
- removed H1: MountingHole_Pad, MountingHole:MountingHole_2.2mm_M2, symbol Mechanical:MountingHole_Pad
- added D1, D2: LED, LED_SMD:LED_0603_1608Metric_Pad1.05x0.95mm_HandSolder, symbol Device:LED
- added R1, R2: R, Resistor_SMD:R_0603_1608Metric_Pad0.98x0.95mm_HandSolder, symbol Device:R
- added U2: 25LC1024 (DIP8 socket), Package_DIP:DIP-8_W7.62mm, symbol Memory_EEPROM:25LCxxx
- added U3: 74HC00, Package_SO:SOIC-14_3.9x8.7mm_P1.27mm, symbol 74xx:74HC00
- C1: footprint Capacitor_SMD:C_0402_1005Metric -> Capacitor_SMD:C_0603_1608Metric_Pad1.08x0.95mm_HandSolder
Connections:
- net +3.3V: now also U2.8 (VCC), U3.14 (VCC)
- net D0: now also U2.5 (MOSI)
- net D1: now also U2.2 (MISO)
- net D2: now also U2.3 (~{WP})
- net D3: now also U2.7 (~{HOLD})
- net GND: now also R1.2, R2.2, U2.4 (GND), U3.10, U3.12, U3.13, U3.7 (GND), U3.9
- net SCK: now also U2.6 (SCK)
- net ~{CS_EEPROM}: now reaches J1.5 (Pin_5)
- net ~{CS_EEPROM}: now also U2.1 (~{CS}), U3.4, U3.5
- net ~{CS} renamed ~{CS_SRAM}
- net ~{CS_SRAM}: now also U3.1, U3.2
- new net: D2.1 (K), R2.1
- new net: D1.1 (K), R1.1
- new net: D1.2 (A), U3.3
- new net: D2.2 (A), U3.6
- no-connect marks 2 -> 1
